File: pcb/base/base.kicad_sch (KiCad schematic)
At the start: 1 part, among them U1 ESP32-S3-WROOM-1-N4R2

Commit message: Finish most of the PCB design
Parts:
- added D1, D2, D3, D4: D_Schottky, symbol Device:D_Schottky
- added J1: Conn_01x03_Pin, symbol Connector:Conn_01x03_Pin
- added J2: Screw_Terminal_01x04, symbol Connector:Screw_Terminal_01x04
- added J3: Screw_Terminal_01x02, symbol Connector:Screw_Terminal_01x02
- added K1, K2, K3, K4: Relay_SPDT, symbol Relay:Relay_SPDT
- added Q1, Q2, Q3, Q4: NMOS, symbol Simulation_SPICE:NMOS
- added R1: 10k, symbol Device:R
- added R2, R3, R4, R5: 330, symbol Device:R
- added R6: 100k, symbol Device:R
- added SW1, SW2: SW_Push, symbol Switch:SW_Push
- added U2: LV2862YDDC, Package_TO_SOT_SMD:SOT-23-6, symbol Regulator_Switching:LV2862YDDC
Connections:
- net GND: now also J1.3 (Pin_3), J3.2 (Pin_2), K1.12, K2.12, K3.12, K4.12, Q1.3 (S), Q2.3 (S), Q3.3 (S), Q4.3 (S), SW1.1, SW2.1, U2.2 (GND)
- net Rail1: now reaches U1.10 (IO17)
- net Rail1: now also J2.1 (Pin_1), K2.11
- net Rail2: now reaches U1.11 (IO18)
- net Rail2: now also J2.2 (Pin_2), K1.11
- net Rail3: now reaches U1.13 (IO19)
- net Rail3: now also J2.3 (Pin_3), K3.11
- net Rail4: now reaches U1.14 (IO20)
- net Rail4: now also J2.4 (Pin_4), K4.11
- net +3V3: now reaches U1.2 (3V3)
- net +3V3: now also R1.1
- net at U1.27 (IO0): now also SW2.2
- net at U1.3 (EN): now also R1.2, SW1.2
- net at U1.36 (RXD0): now also J1.1 (Pin_1)
- net at U1.37 (TXD0): now also J1.2 (Pin_2)
- new net: Q4.2 (G), R5.2
- new net: D2.2 (A), K1.A2, Q2.1 (D)
- new net: R6.2, U2.4 (~{SHDN})
- new net: Q2.2 (G), R3.2
- new net: D3.2 (A), K3.A2, Q3.1 (D)
- new net: D1.2 (A), K2.A2, Q1.1 (D)
- new net: D4.2 (A), K4.A2, Q4.1 (D)
- new net: Q3.2 (G), R4.2
- new net: Q1.2 (G), R2.2
- new net +48V: D1.1 (K), D2.1 (K), D3.1 (K), D4.1 (K), J3.1 (Pin_1), K1.14, K1.A1, K2.14, K2.A1, K3.14, K3.A1, K4.14, K4.A1, R6.1, U2.5 (VIN)
- new net Rail1_Relay: R2.1
- new net Rail2_Relay: R3.1
- new net Rail3_Relay: R4.1
- new net Rail4_Relay: R5.1
