File: pcb/base/base.kicad_sch (KiCad schematic)
At the start: 32 parts, among them J1 Conn_01x03_Pin, J2 Screw_Terminal_01x04, J3 Screw_Terminal_01x02, K1 Relay_SPDT, K2 Relay_SPDT, K3 Relay_SPDT, K4 Relay_SPDT, Q1 NMOS, Q2 NMOS, Q3 NMOS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

Commit message: Finish schematic, add footprints
Parts:
- added C4: 22uF, Capacitor_SMD:C_0805_2012Metric_Pad1.18x1.45mm_HandSolder, symbol Device:C
- added C5: 0.1uF, Capacitor_SMD:C_0805_2012Metric_Pad1.18x1.45mm_HandSolder, symbol Device:C
- C1, C2, C3: footprint (none) -> Capacitor_SMD:C_0805_2012Metric_Pad1.18x1.45mm_HandSolder
- D1, D2, D3, D4: footprint (none) -> footprints:SMAFLAT_STPS2170AF_STM
- D5: footprint (none) -> footprints:DIO_DFLS1100-7
- J1: footprint (none) -> Connector_PinHeader_2.54mm:PinHeader_1x03_P2.54mm_Vertical
- J2: footprint (none) -> footprints:TE_282836-4
- J3: footprint (none) -> footprints:TE_282836-2
- K1, K2, K3, K4: footprint (none) -> footprints:RELAY_PR25-48V-S-360-1C-E
- L1: footprint (none) -> footprints:IND_TAIYO_NR8040_TAY
- Q1, Q2, Q3, Q4: footprint (none) -> Package_TO_SOT_SMD:SOT-523
- R1, R2, R3, R4, R5, R6, R7, R8: footprint (none) -> Resistor_SMD:R_0805_2012Metric_Pad1.20x1.40mm_HandSolder
- SW1, SW2: footprint (none) -> footprints:PTS647SK38SMTR2LFS_CNK
Connections:
- net +3V3: now also C4.1, C5.1
- net GND: now also C4.2, C5.2

Commit message: Finish PCB design
Parts:
- renumbered K2 to K1, K1 to K2
Connections:
- net +3V3: now also R7.1
- net Rail1: no longer U1.10 (IO17)
- net Rail1_Relay: now also U1.10 (IO17)
- net Rail2: no longer U1.11 (IO18)
- net Rail2_Relay: now also U1.11 (IO18)
- net Rail3: no longer U1.13 (IO19)
- net Rail3_Relay: now also U1.13 (IO19)
- net Rail4: no longer U1.14 (IO20)
- net Rail4_Relay: now also U1.14 (IO20)
- net at C1.2, D5.1 (K), L1.1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: no longer R7.1
Other:
- moved on the sheet: L1
Changed lines of the file:
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@@
 	(wire
 		(pts
-			(xy 166.37 67.31) (xy 170.18 67.31)
+			(xy 35.56 128.27) (xy 46.99 128.27)
 		)
 		(stroke
@@
 	(wire
 		(pts
-			(xy 35.56 128.27) (xy 46.99 128.27)
+			(xy 91.44 71.12) (xy 91.44 73.66)
 		)
 		(stroke
@@
 	(wire
 		(pts
-			(xy 91.44 71.12) (xy 91.44 73.66)
+			(xy 151.13 64.77) (xy 151.13 67.31)
 		)
 		(stroke
@@
 	(wire
 		(pts
-			(xy 151.13 64.77) (xy 151.13 67.31)
+			(xy 124.46 77.47) (xy 124.46 80.01)
 		)
 		(stroke
@@
 	(wire
 		(pts
-			(xy 124.46 77.47) (xy 124.46 80.01)
+			(xy 151.13 67.31) (xy 156.21 67.31)
 		)
 		(stroke
@@
 	(wire
 		(pts
-			(xy 151.13 67.31) (xy 166.37 67.31)
-		)
-		(stroke
-			(width 0)
-			(type default)
-		)
-	)
-	(wire
-		(pts
 			(xy 182.88 67.31) (xy 186.69 67.31)
 		)
@@
 	(wire
 		(pts
-			(xy 166.37 67.31) (xy 166.37 71.12)
-		)
-		(stroke
-			(width 0)
-			(type default)
-		)
-	)
-	(wire
-		(pts
 			(xy 59.69 76.2) (xy 59.69 80.01)
 		)
@@
 	(wire
 		(pts
+			(xy 166.37 67.31) (xy 182.88 67.31)
+		)
+		(stroke
+			(width 0)
+			(type default)
+		)
+	)
+	(wire
+		(pts
 			(xy 107.95 125.73) (xy 119.38 125.73)
 		)
@@
 	(wire
 		(pts
-			(xy 177.8 67.31) (xy 182.88 67.31)
+			(xy 166.37 67.31) (xy 166.37 71.12)
 		)
 		(stroke
@@
 	(wire
 		(pts
+			(xy 163.83 67.31) (xy 166.37 67.31)
+		)
+		(stroke
+			(width 0)
+			(type default)
+		)
+	)
+	(wire
+		(pts
 			(xy 143.51 62.23) (xy 143.51 52.07)
 		)
@@
 		)
 	)
-	(label "Rail3"
+	(label "Rail3_Relay"
 		(at 267.97 50.8 0)
 		(effects
@@
 		)
 	)
-	(label "Rail1"
+	(label "Rail1_Relay"
 		(at 267.97 45.72 0)
 		(effects
@@
 		)
 	)
-	(label "Rail4"
+	(label "Rail4_Relay"
 		(at 267.97 53.34 0)
 		(effects
@@
 		)
 	)
-	(label "Rail2"
+	(label "Rail2_Relay"
 		(at 267.97 48.26 0)
 		(effects
@@
 		(dnp no)
 		(fields_autoplaced yes)
-		(property "Reference" "K1"
+		(property "Reference" "K2"
 			(at 63.5 86.3599 0)
 			(effects
@@
 			(project "base"
 				(path "/120457c1-b84d-4e76-b44e-b75b3fe21f22"
-					(reference "K1")
+					(reference "K2")
 					(unit 1)
 				)
@@
 	(symbol
 		(lib_id "Device:L")
-		(at 173.99 67.31 90)
+		(at 160.02 67.31 90)
 		(unit 1)
 		(exclude_from_sim no)
@@
 		(dnp no)
 		(property "Reference" "L1"
-			(at 173.99 62.23 90)
+			(at 160.02 62.23 90)
 			(effects
 				(font
@@
 		)
 		(property "Value" "22uH"
-			(at 173.99 64.77 90)
+			(at 160.02 64.77 90)
 			(effects
 				(font
@@
 		)
 		(property "Footprint" "footprints:IND_TAIYO_NR8040_TAY"
-			(at 173.99 67.31 0)
+			(at 160.02 67.31 0)
 			(effects
 				(font
@@
 		)
 		(property "Datasheet" "~"
-			(at 173.99 67.31 0)
+			(at 160.02 67.31 0)
 			(effects
 				(font
@@
 		)
 		(property "Description" "Inductor"
-			(at 173.99 67.31 0)
+			(at 160.02 67.31 0)
 			(effects
 				(font
@@
 		(dnp no)
 		(fields_autoplaced yes)
-		(property "Reference" "K2"
+		(property "Reference" "K1"
 			(at 63.5 36.8299 0)
 			(effects
@@
 			(project ""
 				(path "/120457c1-b84d-4e76-b44e-b75b3fe21f22"
-					(reference "K2")
+					(reference "K1")
 					(unit 1)
 				)
