File: pcb/base/base.kicad_pcb (KiCad board)
At the start: 2 copper layers, 34 parts, among them J1 Conn_01x03_Pin, J2 Screw_Terminal_01x04, J3 Screw_Terminal_01x02, K1 Relay_SPDT, K2 Relay_SPDT, K3 Relay_SPDT, K4 Relay_SPDT, Q1 NMOS, Q2 NMOS, Q3 NMOS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

Commit message: Finish PCB design
Parts:
- added REF**: MountingHole_5.3mm_M5_Pad, MountingHole:MountingHole_5.3mm_M5_Pad, F.Cu at (140.0, 90.0)
- added REF**: MountingHole_5.3mm_M5_Pad, MountingHole:MountingHole_5.3mm_M5_Pad, F.Cu at (80.0, 170.0)
- added REF**: MountingHole_5.3mm_M5_Pad, MountingHole:MountingHole_5.3mm_M5_Pad, F.Cu at (140.0, 170.0)
- added REF**: MountingHole_5.3mm_M5_Pad, MountingHole:MountingHole_5.3mm_M5_Pad, F.Cu at (80.0, 90.0)
- moved R1 141.3 mm to (78.0, 162.0), turned to 180 degrees
- moved R2 139.4 mm to (104.0, 172.0), turned to -90 degrees
- moved R3 120.1 mm to (104.0, 155.0), turned to -90 degrees
- moved K1 115.4 mm to (121.0, 171.0), turned to 180 degrees
- moved K2 115.1 mm to (121.0, 154.0), turned to 180 degrees
- moved U1 109.0 mm to (83.7, 146.8), turned to 90 degrees
- moved R4 101.1 mm to (104.0, 138.0), turned to -90 degrees
- moved D1 99.8 mm to (108.0, 171.0), turned to -90 degrees
- moved Q1 98.9 mm to (108.4, 176.0), turned to 180 degrees
- moved SW1 97.3 mm to (84.0, 160.6), turned to 180 degrees
- moved C4 88.6 mm to (78.0, 160.0), turned to 180 degrees
- moved C5 84.9 mm to (78.0, 158.0), turned to 180 degrees
- moved R5 82.5 mm to (104.0, 121.0), turned to -90 degrees
- moved Q2 78.4 mm to (108.4, 159.0), turned to 180 degrees
- moved D2 78.3 mm to (108.0, 154.0), turned to -90 degrees
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- renumbered K2 to K1, K1 to K2
Connections:
- R7 pad 1: Net-(D5-K) -> +3V3
- U1 pad 10: /Rail1 -> /Rail1_Relay
- U1 pad 11: /Rail2 -> /Rail2_Relay
- U1 pad 13: /Rail3 -> /Rail3_Relay
- U1 pad 14: /Rail4 -> /Rail4_Relay
Routing:
- net +3V3: track 0.00 -> 134.8 mm, vias 0 -> 2
- net +48V: track 0.00 -> 78.1 mm
- net GND: track 0.00 -> 65.9 mm, vias 0 -> 11
- net /Rail4_Relay: track 0.00 -> 47.4 mm
- net /Rail1: track 0.00 -> 47.2 mm
- net /Rail2: track 0.00 -> 37.8 mm
- net /Rail3_Relay: track 0.00 -> 33.5 mm
- net /Rail3: track 0.00 -> 27.8 mm
- net Net-(D4-A): track 0.00 -> 26.2 mm
- net Net-(D3-A): track 0.00 -> 25.4 mm
- net Net-(D1-A): track 0.00 -> 25.1 mm
- net Net-(D2-A): track 0.00 -> 25.1 mm
- net /Rail1_Relay: track 0.00 -> 21.4 mm
- net /Rail2_Relay: track 0.00 -> 19.6 mm
- net /Rail4: track 0.00 -> 18.9 mm
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- added copper zone on B.Cu, net +48V
- added copper zone on B.Cu, net GND
- added copper zone on F.Cu, net Net-(D5-K)
Other:
- board outline added: 80 x 100 mm
